Commit message: update 26/6

File: install/go1_description/share/go1_description/xacro/robot.xacro (robot description, xacro)
@@ -9,8 +9,21 @@
     <xacro:include filename="$(find go1_description)/xacro/materials.xacro"/>
     <xacro:include filename="$(find go1_description)/xacro/leg.xacro"/>
+    <!-- <xacro:include filename="$(find go1_description)/xacro/stairs.xacro"/> -->
     <xacro:include filename="$(find go1_description)/xacro/gazebo.xacro"/>
     <xacro:include filename="$(find go1_description)/xacro/depthCamera.xacro"/>
     <xacro:include filename="$(find go1_description)/xacro/ultraSound.xacro"/>
-    <xacro:include filename="$(find go1_description)/xacro/transmission.xacro"/>
+    <!-- <xacro:include filename="$(find go1_gazebo)/launch/stairs.urdf.xacro"/> -->
+    <!-- <xacro:stairs stairs="15" xpos="0" ypos="0" zpos="0" /> -->
+    <!-- Rotor related joint and link is only for demonstrate location. -->
+    <!-- Actually, the rotor will rotate and the joint is not fixed. Reduction ratio should be considered. -->
+    <!-- Debug mode will hung up the robot, use "true" or "false" to switch it. -->
+    <!-- <xacro:if value="$(arg DEBUG)">
+        <link name="world"/>
+        <joint name="base_static_joint" type="fixed">
+            <origin rpy="0 0 0" xyz="0 0 0"/>
+            <parent link="world"/>
+            <child link="base"/>
+        </joint>
+    </xacro:if>  -->
     <link name="base">
         <visual>
@@ -22,5 +35,5 @@
     </link>
     <xacro:if value="$(arg use_nav2_links)">
-        <link name="base_link"/>
+        <link name="base_link" />
         <joint name="base_link_to_base" type="fixed">
             <origin rpy="0 0 0" xyz="0 0 0"/>
@@ -28,5 +41,6 @@
             <child link="base"/>
         </joint>
-        <link name="height_measurement"/>
+        <link name="height_measurement" />
+        <!-- Measured empirically from difference between actual and reported body height -->
         <joint name="base_link_to_height" type="fixed">
             <origin rpy="0 0 0" xyz="0 0 -0.015"/>
@@ -34,14 +48,15 @@
             <child link="height_measurement"/>
         </joint>
-        <link name="base_footprint"/>
+        <link name="base_footprint" />
         <joint name="height_to_footprint" type="prismatic">
-            <parent link="height_measurement"/>
-            <child link="base_footprint"/>
-            <origin xyz="0 0 0" rpy="0 0 0"/>
-            <axis xyz="0 0 -1"/>
-            <limit effort="100000.0" lower="0.0" upper="1.0" velocity="100000.0"/>
+                <parent link="height_measurement"/>
+                <child link="base_footprint"/>
+                <origin xyz = "0 0 0" rpy="0 0 0"/>
+                <axis xyz="0 0 -1" />
+                <limit effort="100000.0" lower="0.0" upper="1.0" velocity="100000.0"/>
         </joint>
-        <link name="base_laser"/>
+        <link name="base_laser" />
         <joint name="base_link_to_lidar" type="fixed">
+            <!-- TODO need to measure mounting or make this a parameter -->
             <origin rpy="0 0 0" xyz="$(arg lidar_x_offset) $(arg lidar_y_offset) $(arg lidar_z_offset)"/>
             <parent link="base_link"/>
@@ -60,4 +75,5 @@
                 <mesh filename="package://go1_description/meshes/trunk.dae" scale="1 1 1"/>
             </geometry>
+            <!-- <material name="orange"/> -->
         </visual>
         <collision>
@@ -92,4 +108,5 @@
                 <box size="0.001 0.001 0.001"/>
             </geometry>
+            <!-- <material name="red"/> -->
         </visual>
         <collision>
@@ -100,8 +117,8 @@
         </collision>
     </link>
-    <xacro:leg name="FR" mirror="-1" mirror_dae="False" front_hind="1" front_hind_dae="True"/>
-    <xacro:leg name="FL" mirror="1" mirror_dae="True" front_hind="1" front_hind_dae="True"/>
-    <xacro:leg name="RR" mirror="-1" mirror_dae="False" front_hind="-1" front_hind_dae="False"/>
-    <xacro:leg name="RL" mirror="1" mirror_dae="True" front_hind="-1" front_hind_dae="False"/>
+    <xacro:leg name="FR" mirror="-1" mirror_dae= "False" front_hind="1"  front_hind_dae="True"  />
+    <xacro:leg name="FL" mirror="1"  mirror_dae="True"   front_hind="1"  front_hind_dae="True"  />
+    <xacro:leg name="RR" mirror="-1" mirror_dae="False"  front_hind="-1" front_hind_dae="False" />
+    <xacro:leg name="RL" mirror="1"  mirror_dae="True"   front_hind="-1" front_hind_dae="False" />
     <xacro:depthCamera camID="1" name="face">
         <origin rpy="${PI} 0 0" xyz="0.2785 0.0125 0.0167"/>
@@ -134,5 +151,5 @@
     </link>
     <xacro:ultraSound name="left">
-        <origin rpy="0 0.2618 ${PI/2}" xyz="-0.0535 0.0826 0.00868"/>
+        <origin rpy="0 0.2618 ${PI/2}" xyz="-0.0535  0.0826 0.00868"/>
     </xacro:ultraSound>
     <xacro:ultraSound name="right">
